File: schematics/VOX_V847.kicad_sch (KiCad schematic)
At the start: 23 parts, among them J1 Stereo Phone Jack, J2 MONO Phone Jack, Q1 MPSA18, Q2 MPSA18, SW1 SW_SPDT

Commit message: Update VOX_V847.kicad_sch
Parts:
- SW1: value SW_SPDT -> SPDT Foot SW
- renumbered R1 to R3
Changed lines of the file:
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@@
 		(on_board yes)
 		(dnp no)
-		(property "Reference" "R1"
+		(property "Reference" "R3"
 			(at 126.238 110.49 90)
 			(effects
@@
 			(project "Wah"
 				(path "/c098d18e-1cd1-4188-b86d-6c575f30bd7b/e57f705d-972f-46c2-991e-b87085ebf6c1"
-					(reference "R1")
+					(reference "R3")
 					(unit 1)
 				)
@@
 		(dnp no)
 		(fields_autoplaced yes)
-		(property "Reference" "C?"
+		(property "Reference" "C1"
 			(at 104.14 88.9 90)
 			(effects
@@
 			(project "Wah"
 				(path "/c098d18e-1cd1-4188-b86d-6c575f30bd7b/e57f705d-972f-46c2-991e-b87085ebf6c1"
-					(reference "C?")
+					(reference "C1")
 					(unit 1)
 				)
@@
 			)
 		)
-		(property "Value" "SW_SPDT"
+		(property "Value" "SPDT Foot SW"
 			(at 215.9 90.17 0)
 			(effects
