File: schematics/VOX_V847_Mod.kicad_sch (KiCad schematic)
At the start: 30 parts, among them J3 Stereo Phone Jack, J4 MONO Phone Jack, J5 Barrel_Jack_Switch, Q3 MPSA18, Q4 MPSA18, SW1 SW_DPDT_x3, SW2 SW_SPDT, SW3 SW_SPDT

Commit message: Update VOX_V847_Mod.kicad_sch
Parts:
- SW1: value SW_DPDT_x3 -> 3PDT Foot SW
- SW2, SW3: value SW_SPDT -> SPDT Toggle
- renumbered BT2 to BT1, C6 to C2, C7 to C3, C8 to C4, C9 to C5, J3 to J1, J4 to J2, J5 to J3, L2 to L1, Q3 to Q1, Q4 to Q2, R16 to R1, R19 to R10, R8 to R2, R15 to R3, R11 to R3, R14 to R4, R13 to R5, R12 to R6, R17 to R7, R18 to R9, RV2 to RV1
Changed lines of the file:
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@@
 		(rev "A")
 		(company "JJ1LFO@jarl.com")
+		(comment 1 "True Bypass")
 		(comment 2 "ON LED")
-		(comment 3 "True Bypass")
+		(comment 3 "True Bypass/Non-True Bypass Switch")
+		(comment 4 "Gain Freq Switch")
 	)
 	(text "Non-TRUE"
@@
 		(dnp no)
 		(property "Reference" "SW1"
-			(at 124.968 76.962 0)
+			(at 128.016 77.216 0)
 			(effects
 				(font
@@
 			)
 		)
-		(property "Value" "SW_DPDT_x3"
-			(at 123.698 79.502 0)
+		(property "Value" "3PDT Foot SW"
+			(at 127.508 79.502 0)
 			(effects
 				(font
@@
 		(on_board yes)
 		(dnp no)
-		(property "Reference" "Q3"
+		(property "Reference" "Q1"
 			(at 138.43 87.884 0)
 			(effects
@@
 			(project "Wah"
 				(path "/c098d18e-1cd1-4188-b86d-6c575f30bd7b/032a59bf-fc15-453b-8cf7-d567bc13a2ae"
-					(reference "Q3")
+					(reference "Q1")
 					(unit 1)
 				)
@@
 		(on_board yes)
 		(dnp no)
-		(property "Reference" "R12"
+		(property "Reference" "R6"
 			(at 141.478 66.04 90)
 			(effects
@@
 			(project "Wah"
 				(path "/c098d18e-1cd1-4188-b86d-6c575f30bd7b/032a59bf-fc15-453b-8cf7-d567bc13a2ae"
-					(reference "R12")
+					(reference "R6")
 					(unit 1)
 				)
@@
 		(on_board yes)
 		(dnp no)
-		(property "Reference" "R13"
+		(property "Reference" "R5"
 			(at 141.478 109.22 90)
 			(effects
@@
 			(project "Wah"
 				(path "/c098d18e-1cd1-4188-b86d-6c575f30bd7b/032a59bf-fc15-453b-8cf7-d567bc13a2ae"
-					(reference "R13")
+					(reference "R5")
 					(unit 1)
 				)
@@
 			)
 		)
-		(property "Value" "SW_DPDT_x3"
+		(property "Value" "3PDT Foot SW"
 			(at 102.108 89.154 0)
 			(effects
@@
 		(on_board yes)
 		(dnp no)
-		(property "Reference" "R17"
+		(property "Reference" "R7"
 			(at 215.138 95.25 90)
 			(effects
@@
 			(project "Wah"
 				(path "/c098d18e-1cd1-4188-b86d-6c575f30bd7b/032a59bf-fc15-453b-8cf7-d567bc13a2ae"
-					(reference "R17")
+					(reference "R7")
 					(unit 1)
 				)
@@
 			)
 		)
-		(property "Value" "SW_SPDT"
+		(property "Value" "SPDT Toggle"
 			(at 144.018 132.08 0)
 			(effects
@@
 		(on_board yes)
 		(dnp no)
-		(property "Reference" "R14"
+		(property "Reference" "R4"
 			(at 151.638 96.52 90)
 			(effects
@@
 			(project "Wah"
 				(path "/c098d18e-1cd1-4188-b86d-6c575f30bd7b/032a59bf-fc15-453b-8cf7-d567bc13a2ae"
-					(reference "R14")
+					(reference "R4")
 					(unit 1)
 				)
@@
 		(on_board yes)
 		(dnp no)
-		(property "Reference" "BT2"
+		(property "Reference" "BT1"
 			(at 50.546 79.248 90)
 			(effects
@@
 			(project "Wah"
 				(path "/c098d18e-1cd1-4188-b86d-6c575f30bd7b/032a59bf-fc15-453b-8cf7-d567bc13a2ae"
-					(reference "BT2")
+					(reference "BT1")
 					(unit 1)
 				)
@@
 		(dnp no)
 		(fields_autoplaced yes)
-		(property "Reference" "J5"
+		(property "Reference" "J3"
 			(at 48.26 48.26 0)
 			(effects
@@
 			(project ""
 				(path "/c098d18e-1cd1-4188-b86d-6c575f30bd7b/032a59bf-fc15-453b-8cf7-d567bc13a2ae"
-					(reference "J5")
+					(reference "J3")
 					(unit 1)
 				)
@@
 		(dnp no)
 		(fields_autoplaced yes)
-		(property "Reference" "R8"
+		(property "Reference" "R2"
 			(at 119.38 88.9 90)
 			(effects
@@
 			(project "Wah"
 				(path "/c098d18e-1cd1-4188-b86d-6c575f30bd7b/032a59bf-fc15-453b-8cf7-d567bc13a2ae"
-					(reference "R8")
+					(reference "R2")
 					(unit 1)
 				)
@@
 			)
 		)
-		(property "Value" "SW_SPDT"
+		(property "Value" "SPDT Toggle"
 			(at 88.9 86.36 0)
 			(effects
@@
 		(on_board yes)
 		(dnp no)
-		(property "Reference" "R19"
+		(property "Reference" "R10"
 			(at 229.108 121.412 90)
 			(effects
@@
 			(project "Wah"
 				(path "/c098d18e-1cd1-4188-b86d-6c575f30bd7b/032a59bf-fc15-453b-8cf7-d567bc13a2ae"
-					(reference "R19")
+					(reference "R10")
 					(unit 1)
 				)
@@
 		(on_board yes)
 		(dnp no)
-		(property "Reference" "R15"
+		(property "Reference" "R3"
 			(at 151.638 109.22 90)
 			(effects
@@
 			(project "Wah"
 				(path "/c098d18e-1cd1-4188-b86d-6c575f30bd7b/032a59bf-fc15-453b-8cf7-d567bc13a2ae"
-					(reference "R15")
+					(reference "R3")
 					(unit 1)
 				)
@@
 		(on_board yes)
 		(dnp no)
-		(property "Reference" "J4"
+		(property "Reference" "J2"
 			(at 252.476 97.79 0)
 			(effects
@@
 			(project "Wah"
 				(path "/c098d18e-1cd1-4188-b86d-6c575f30bd7b/032a59bf-fc15-453b-8cf7-d567bc13a2ae"
-					(reference "J4")
+					(reference "J2")
 					(unit 1)
 				)
@@
 		(on_board yes)
 		(dnp no)
-		(property "Reference" "R18"
+		(property "Reference" "R9"
 			(at 229.108 89.662 90)
 			(effects
@@
 			(project "Wah"
 				(path "/c098d18e-1cd1-4188-b86d-6c575f30bd7b/032a59bf-fc15-453b-8cf7-d567bc13a2ae"
-					(reference "R18")
+					(reference "R9")
 					(unit 1)
 				)
@@
 		(on_board yes)
 		(dnp no)
-		(property "Reference" "C6"
+		(property "Reference" "C2"
 			(at 160.02 108.966 90)
 			(effects
@@
 			(project "Wah"
 				(path "/c098d18e-1cd1-4188-b86d-6c575f30bd7b/032a59bf-fc15-453b-8cf7-d567bc13a2ae"
-					(reference "C6")
+					(reference "C2")
 					(unit 1)
 				)
@@
 		(on_board yes)
 		(dnp no)
-		(property "Reference" "L2"
+		(property "Reference" "L1"
 			(at 178.816 110.236 90)
 			(effects
@@
 			(project "Wah"
 				(path "/c098d18e-1cd1-4188-b86d-6c575f30bd7b/032a59bf-fc15-453b-8cf7-d567bc13a2ae"
-					(reference "L2")
+					(reference "L1")
 					(unit 1)
 				)
@@
 		(on_board yes)
 		(dnp no)
-		(property "Reference" "R11"
+		(property "Reference" "R3"
 			(at 131.318 102.87 90)
 			(effects
@@
 			(project "Wah"
 				(path "/c098d18e-1cd1-4188-b86d-6c575f30bd7b/032a59bf-fc15-453b-8cf7-d567bc13a2ae"
-					(reference "R11")
+					(reference "R3")
 					(unit 1)
 				)
@@
 		(on_board yes)
 		(dnp no)
-		(property "Reference" "C9"
+		(property "Reference" "C5"
 			(at 210.566 92.456 90)
 			(effects
@@
 			(project "Wah"
 				(path "/c098d18e-1cd1-4188-b86d-6c575f30bd7b/032a59bf-fc15-453b-8cf7-d567bc13a2ae"
-					(reference "C9")
+					(reference "C5")
 					(unit 1)
 				)
@@
 			)
 		)
-		(property "Value" "SW_DPDT_x3"
+		(property "Value" "3PDT Foot SW"
 			(at 241.808 88.9 0)
 			(effects
@@
 		(on_board yes)
 		(dnp no)
-		(property "Reference" "Q4"
+		(property "Reference" "Q2"
 			(at 226.06 91.694 0)
 			(effects
@@
 			(project "Wah"
 				(path "/c098d18e-1cd1-4188-b86d-6c575f30bd7b/032a59bf-fc15-453b-8cf7-d567bc13a2ae"
-					(reference "Q4")
+					(reference "Q2")
 					(unit 1)
 				)
@@
 		(on_board yes)
 		(dnp no)
-		(property "Reference" "C8"
+		(property "Reference" "C4"
 			(at 190.246 117.856 90)
 			(effects
@@
 			(project "Wah"
 				(path "/c098d18e-1cd1-4188-b86d-6c575f30bd7b/032a59bf-fc15-453b-8cf7-d567bc13a2ae"
-					(reference "C8")
+					(reference "C4")
 					(unit 1)
 				)
@@
 		(on_board yes)
 		(dnp no)
-		(property "Reference" "R16"
-			(at 170.688 110.49 90)
+		(property "Reference" "R1"
+			(at 170.688 111.252 90)
 			(effects
 				(font
@@
 			(project "Wah"
 				(path "/c098d18e-1cd1-4188-b86d-6c575f30bd7b/032a59bf-fc15-453b-8cf7-d567bc13a2ae"
-					(reference "R16")
+					(reference "R1")
 					(unit 1)
 				)
@@
 		(on_board yes)
 		(dnp no)
-		(property "Reference" "J3"
+		(property "Reference" "J1"
 			(at 46.99 90.678 0)
 			(effects
@@
 			(project "Wah"
 				(path "/c098d18e-1cd1-4188-b86d-6c575f30bd7b/032a59bf-fc15-453b-8cf7-d567bc13a2ae"
-					(reference "J3")
+					(reference "J1")
 					(unit 1)
 				)
@@
 		(on_board yes)
 		(dnp no)
-		(property "Reference" "RV2"
+		(property "Reference" "RV1"
 			(at 186.182 100.33 90)
 			(effects
@@
 			(project "Wah"
 				(path "/c098d18e-1cd1-4188-b86d-6c575f30bd7b/032a59bf-fc15-453b-8cf7-d567bc13a2ae"
-					(reference "RV2")
+					(reference "RV1")
 					(unit 1)
 				)
@@
 		(on_board yes)
 		(dnp no)
-		(property "Reference" "C7"
+		(property "Reference" "C3"
 			(at 182.372 74.676 90)
 			(effects
@@
 			(project "Wah"
 				(path "/c098d18e-1cd1-4188-b86d-6c575f30bd7b/032a59bf-fc15-453b-8cf7-d567bc13a2ae"
-					(reference "C7")
+					(reference "C3")
 					(unit 1)
 				)

Commit message: Update VOX_V847_Mod.kicad_sch
Connections:
- net Earth: now also SW3.2 (B); no longer R21.1
- net at Q1.1 (E), R5.2: now also R21.2; no longer SW3.2 (B)
- net at SW3.3 (C): now also R21.1; no longer R21.2
Other:
- moved on the sheet: R21, SW3
Changed lines of the file:
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@@
 	(text_box "Increase gain and lower heel-side frequency."
 		(exclude_from_sim no)
-		(at 156.21 129.54 0)
+		(at 163.83 129.54 0)
 		(size 26.67 6.35)
 		(margins 0.9525 0.9525 0.9525 0.9525)
@@
 	)
 	(no_connect
-		(at 147.32 137.16)
+		(at 154.94 138.43)
 	)
 	(wire
@@
 	(wire
 		(pts
-			(xy 152.4 137.16) (xy 152.4 138.43)
-		)
-		(stroke
-			(width 0)
-			(type default)
-		)
-	)
-	(wire
-		(pts
 			(xy 166.37 104.14) (xy 166.37 101.6)
 		)
@@
 	(wire
 		(pts
-			(xy 152.4 146.05) (xy 152.4 147.32)
-		)
-		(stroke
-			(width 0)
-			(type default)
-		)
-	)
-	(wire
-		(pts
 			(xy 250.19 104.14) (xy 247.65 104.14)
 		)
@@
 	(wire
 		(pts
+			(xy 149.86 134.62) (xy 149.86 138.43)
+		)
+		(stroke
+			(width 0)
+			(type default)
+		)
+	)
+	(wire
+		(pts
 			(xy 146.05 111.76) (xy 146.05 113.03)
 		)
@@
 		(pts
 			(xy 184.15 105.41) (xy 184.15 101.6)
+		)
+		(stroke
+			(width 0)
+			(type default)
+		)
+	)
+	(wire
+		(pts
+			(xy 152.4 148.59) (xy 152.4 151.13)
 		)
 		(stroke
@@
 		(dnp no)
 		(property "Reference" "SW1"
-			(at 128.016 77.216 0)
+			(at 127.762 76.454 0)
 			(effects
 				(font
@@
 		)
 		(property "Value" "3PDT Foot SW"
-			(at 127.508 79.502 0)
+			(at 125.222 79.502 0)
 			(effects
 				(font
@@
 	(symbol
 		(lib_id "power:GND")
-		(at 152.4 147.32 0)
+		(at 152.4 151.13 0)
 		(unit 1)
 		(exclude_from_sim no)
@@
 		(fields_autoplaced yes)
 		(property "Reference" "#PWR016"
-			(at 152.4 153.67 0)
+			(at 152.4 157.48 0)
 			(effects
 				(font
@@
 		)
 		(property "Value" "GND"
-			(at 152.4 152.4 0)
+			(at 152.4 156.21 0)
 			(effects
 				(font
@@
 		)
 		(property "Footprint" ""
-			(at 152.4 147.32 0)
+			(at 152.4 151.13 0)
 			(effects
 				(font
@@
 		)
 		(property "Datasheet" ""
-			(at 152.4 147.32 0)
+			(at 152.4 151.13 0)
 			(effects
 				(font
@@
 		)
 		(property "Description" "Power symbol creates a global label with name \"GND\" , ground"
-			(at 152.4 147.32 0)
+			(at 152.4 151.13 0)
 			(effects
 				(font
@@
 	(symbol
 		(lib_id "Switch:SW_SPDT")
-		(at 149.86 132.08 90)
+		(at 152.4 143.51 270)
 		(mirror x)
 		(unit 1)
@@
 		(dnp no)
 		(property "Reference" "SW3"
-			(at 141.986 132.334 0)
+			(at 160.274 143.256 0)
 			(effects
 				(font
@@
 		)
 		(property "Value" "SPDT Toggle"
-			(at 144.018 132.08 0)
+			(at 158.242 143.51 0)
 			(effects
 				(font
@@
 		)
 		(property "Footprint" ""
-			(at 149.86 132.08 0)
+			(at 152.4 143.51 0)
 			(effects
 				(font
@@
 		)
 		(property "Datasheet" "~"
-			(at 157.48 132.08 0)
+			(at 144.78 143.51 0)
 			(effects
 				(font
@@
 		)
 		(property "Description" "Switch, single pole double throw"
-			(at 149.86 132.08 0)
+			(at 152.4 143.51 0)
 			(effects
 				(font
@@
 	(symbol
 		(lib_id "Device:R")
-		(at 152.4 142.24 180)
+		(at 149.86 130.81 180)
 		(unit 1)
 		(exclude_from_sim no)
@@
 		(dnp no)
 		(property "Reference" "R21"
-			(at 147.828 143.51 90)
+			(at 145.288 132.08 90)
 			(effects
 				(font
@@
 		)
 		(property "Value" "1k5"
-			(at 149.86 144.018 90)
+			(at 147.32 132.588 90)
 			(effects
 				(font
@@
 		)
 		(property "Footprint" ""
-			(at 154.178 142.24 90)
+			(at 151.638 130.81 90)
 			(effects
 				(font
@@
 		)
 		(property "Datasheet" "~"
-			(at 152.4 142.24 0)
+			(at 149.86 130.81 0)
 			(effects
 				(font
@@
 		)
 		(property "Description" "Resistor"
-			(at 152.4 142.24 0)
-			(effects
-				(font
+			(at 149.86 130.81 0)
+			(effects
+				(font

Commit message: Update VOX_V847_Mod.kicad_sch
Parts:
- renumbered D2 to D1, D1 to D2, J3 to J1, J1 to J2, J2 to J3, R20 to R1, R9 to R10, R10 to R11, R6 to R4, R4 to R6, R3 to R7, R1 to R8, R7 to R9, R21 to R?
Connections:
- net BLUE: now also SW1.7 (A); no longer SW1.1 (A)
- net BROWN: now also SW1.2 (B); no longer SW1.5 (B)
- net Earth: now also SW1.5 (B), SW1.6 (C), SW1.8 (B); no longer SW1.2 (B), SW1.8 (B), SW1.9 (C)
- net GREEN: now also SW1.1 (A), SW1.9 (C); no longer SW1.3 (C), SW1.4 (A)
- net at D2.1 (K): now also SW1.4 (A); no longer SW1.7 (A)
- net at SW2.2 (B): now also SW1.3 (C); no longer SW1.6 (C)
Changed lines of the file:
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@@
 		(lib_id "Switch:SW_DPDT_x2")
 		(at 128.27 69.85 180)
-		(unit 3)
+		(unit 2)
 		(exclude_from_sim no)
 		(in_bom yes)
@@
 			(project "VOX_V847_Mod"
 				(path "/9e37ffa3-1d98-44a8-bc9d-bb74969d79c6"
-					(reference "SW3")
-					(unit 1)
+					(reference "SW1")
+					(unit 2)
 				)
 			)
@@
 		(dnp no)
 		(fields_autoplaced yes)
-		(property "Reference" "#PWR016"
+		(property "Reference" "#PWR?"
 			(at 152.4 157.48 0)
 			(effects
@@
 		)
 		(instances
+			(project "VOX_V847_Mod"
+				(path "/9e37ffa3-1d98-44a8-bc9d-bb74969d79c6"
+					(reference "#PWR?")
+					(unit 1)
+				)
+			)
 			(project "Wah"
 				(path "/c098d18e-1cd1-4188-b86d-6c575f30bd7b/032a59bf-fc15-453b-8cf7-d567bc13a2ae"
@@
 		(on_board yes)
 		(dnp no)
-		(property "Reference" "R6"
+		(property "Reference" "R4"
 			(at 141.478 66.04 90)
 			(effects
@@
 		(lib_id "Switch:SW_DPDT_x2")
 		(at 102.87 95.25 180)
-		(unit 2)
+		(unit 1)
 		(exclude_from_sim no)
 		(in_bom yes)
@@
 			(project "VOX_V847_Mod"
 				(path "/9e37ffa3-1d98-44a8-bc9d-bb74969d79c6"
-					(reference "SW2")
+					(reference "SW1")
 					(unit 1)
 				)
@@
 		(on_board yes)
 		(dnp no)
-		(property "Reference" "R7"
+		(property "Reference" "R9"
 			(at 215.138 95.25 90)
 			(effects
@@
 		)
 		(instances
+			(project "VOX_V847_Mod"
+				(path "/9e37ffa3-1d98-44a8-bc9d-bb74969d79c6"
+					(reference "SW3")
+					(unit 1)
+				)
+			)
 			(project "Wah"
 				(path "/c098d18e-1cd1-4188-b86d-6c575f30bd7b/032a59bf-fc15-453b-8cf7-d567bc13a2ae"
@@
 		(on_board yes)
 		(dnp no)
-		(property "Reference" "R4"
+		(property "Reference" "R6"
 			(at 151.638 96.52 90)
 			(effects
@@
 		(dnp no)
 		(fields_autoplaced yes)
-		(property "Reference" "#PWR013"
+		(property "Reference" "#PWR07"
 			(at 233.68 130.81 0)
 			(effects
@@
 		(dnp no)
 		(fields_autoplaced yes)
-		(property "Reference" "J3"
+		(property "Reference" "J1"
 			(at 48.26 48.26 0)
 			(effects
@@
 		(on_board yes)
 		(dnp no)
-		(property "Reference" "D1"
+		(property "Reference" "D2"
 			(at 114.808 65.786 0)
 			(effects
@@
 			(project ""
 				(path "/9e37ffa3-1d98-44a8-bc9d-bb74969d79c6"
-					(reference "SW1")
+					(reference "SW2")
 					(unit 1)
 				)
@@
 		(on_board yes)
 		(dnp no)
-		(property "Reference" "R10"
+		(property "Reference" "R11"
 			(at 229.108 121.412 90)
 			(effects
@@
 		(on_board yes)
 		(dnp no)
-		(property "Reference" "R20"
+		(property "Reference" "R1"
 			(at 100.584 68.072 90)
 			(effects
@@
 		(on_board yes)
 		(dnp no)
-		(property "Reference" "R3"
+		(property "Reference" "R7"
 			(at 151.638 109.22 90)
 			(effects
@@
 		(on_board yes)
 		(dnp no)
-		(property "Reference" "J2"
+		(property "Reference" "J3"
 			(at 252.476 97.79 0)
 			(effects
@@
 		(dnp no)
 		(fields_autoplaced yes)
-		(property "Reference" "#PWR014"
+		(property "Reference" "#PWR08"
 			(at 247.65 115.57 0)
 			(effects
@@
 		(on_board yes)
 		(dnp no)
-		(property "Reference" "R9"
+		(property "Reference" "R10"
 			(at 229.108 89.662 90)
 			(effects
@@
 		(on_board yes)
 		(dnp no)
-		(property "Reference" "R21"
+		(property "Reference" "R?"
 			(at 145.288 132.08 90)
 			(effects
@@
 		)
 		(instances
+			(project "VOX_V847_Mod"
+				(path "/9e37ffa3-1d98-44a8-bc9d-bb74969d79c6"
+					(reference "R?")
+					(unit 1)
+				)
+			)
 			(project "Wah"
 				(path "/c098d18e-1cd1-4188-b86d-6c575f30bd7b/032a59bf-fc15-453b-8cf7-d567bc13a2ae"
@@
 		(dnp no)
 		(fields_autoplaced yes)
-		(property "Reference" "#PWR011"
+		(property "Reference" "#PWR05"
 			(at 156.21 119.38 0)
 			(effects
@@
 		(dnp no)
 		(fields_autoplaced yes)
-		(property "Reference" "#PWR09"
+		(property "Reference" "#PWR02"
 			(at 81.28 113.03 0)
 			(effects
@@
 		(dnp no)
 		(fields_autoplaced yes)
-		(property "Reference" "#PWR010"
+		(property "Reference" "#PWR04"
 			(at 146.05 119.38 0)
 			(effects
@@
 		(lib_id "Switch:SW_DPDT_x2")
 		(at 247.65 88.9 90)
-		(unit 1)
+		(unit 3)
 		(exclude_from_sim no)
 		(in_bom yes)
@@
 			(project "VOX_V847_Mod"
 				(path "/9e37ffa3-1d98-44a8-bc9d-bb74969d79c6"
-					(reference "SW4")
-					(unit 1)
+					(reference "SW1")
+					(unit 3)
 				)
 			)
@@
 		(dnp no)
 		(fields_autoplaced yes)
-		(property "Reference" "#PWR015"
+		(property "Reference" "#PWR?"
 			(at 134.62 80.01 0)
 			(effects
@@
 		)
 		(instances
+			(project "VOX_V847_Mod"
+				(path "/9e37ffa3-1d98-44a8-bc9d-bb74969d79c6"
+					(reference "#PWR?")
+					(unit 1)
+				)
+			)
 			(project "Wah"
 				(path "/c098d18e-1cd1-4188-b86d-6c575f30bd7b/032a59bf-fc15-453b-8cf7-d567bc13a2ae"
@@
 		(on_board yes)
 		(dnp no)
-		(property "Reference" "R1"
+		(property "Reference" "R8"
 			(at 170.688 111.252 90)
 			(effects
@@
 		(on_board yes)
 		(dnp no)
-		(property "Reference" "J1"
+		(property "Reference" "J2"
 			(at 46.99 90.678 0)
 			(effects
@@
 		(on_board yes)
 		(dnp no)
-		(property "Reference" "D2"
+		(property "Reference" "D1"
 			(at 108.204 75.184 0)
 			(effects
@@
 		(dnp no)
 		(fields_autoplaced yes)
-		(property "Reference" "#PWR012"
+		(property "Reference" "#PWR06"
 			(at 166.37 119.38 0)
 			(effects
@@
 		(dnp no)
 		(fields_autoplaced yes)
-		(property "Reference" "#PWR06"
+		(property "Reference" "#PWR01"
 			(at 57.15 113.03 0)
 			(effects
