File: schematics/VOX_V847_Mod.kicad_sch (KiCad schematic)
At the start: 30 parts, among them J1 Barrel_Jack_Switch, J2 Stereo Phone Jack, J3 MONO Phone Jack, Q1 MPSA18, Q2 MPSA18, SW1 3PDT Foot SW, SW2 SPDT Toggle, SW3 SPDT Toggle

Commit message: Update VOX_V847_Mod.kicad_sch
Parts:
- added D3: 1N4001, Diode_THT:D_DO-41_SOD81_P10.16mm_Horizontal, symbol Diode:1N4001
Connections:
- net Earth: now also D3.2 (A)
- net RED: now also D3.1 (K)
Other:
- moved on the sheet: BT1, J1, J2
